File: Hardware/particle-logo-v1.brd (EAGLE design)
At the start: 76.2 x 27.9 mm, 17 parts, among them U1 USD-SOCKETMOLEX-CORRECT, U2 APDS-9960

Commit message: Add BOM and schematics PDF
Parts:
- renumbered U$2 to U3, U$8 to U4
