File: Hardware/particle-logo-v1.sch (EAGLE design)
At the start: 17 parts, among them U1 USD-SOCKETMOLEX-CORRECT, U2 APDS-9960

Commit message: Add BOM and schematics PDF
Parts:
- C1: PARTNO (none) -> EEU-FR1C102L
- C2: PARTNO (none) -> 0603YD105KAT2A
- C3: PARTNO (none) -> CC0603JRX7R7BB104
- C4: PARTNO (none) -> TAJD107K020RNJ
- R1, R3: PARTNO (none) -> ERJ-3EKF1002V
- R2: PARTNO (none) -> ERJ-3GEYJ221V
- R4: DNP (none) -> t
- STANDOFF1, STANDOFF2, U$1: BOM (none) -> exclude
- U1: PARTNO (none) -> 1040310811
- U2: PARTNO (none) -> APDS-9960
- U4: PARTNO (none) -> NL17SZ125DTT1G
- renumbered U$2 to U3, U$8 to U4
